Commit message: added inertia properties

File: data/urdf/tests/test_merge_joints.urdf (robot description, URDF)
Before this commit: robot test_merge_joints, 5 links, 4 joints
Joints:
- joint elbow_joint: origin xyz=0 0 0.4 -> xyz=0 0 0.4 rpy=1.571 0. 0.

Commit message: changed test_merge_joints.urdf to match with test_basic.urdf, except two fixed joints

File: data/urdf/tests/test_merge_joints.urdf (robot description, URDF)
Before this commit: robot test_merge_joints, 5 links, 4 joints
Links:
- added link finger_link_1; collision box size=0.06 .1 .1; visual box size=0.06 .01 .01
- added link finger_link_2; collision box size=0.06 .1 .1; visual box size=0.06 .01 .01
Joints:
- added joint finger_1_joint: type prismatic, parent palm_link, child finger_link_1, origin xyz=-0.10 0 0.05 rpy=0 1.571 0, axis 0 0 1, limit lower=-0.02 upper=0.08 effort=1000.0 velocity=0.5
- added joint finger_2_joint: type prismatic, parent palm_link, child finger_link_2, origin xyz=0.10 0 0.05 rpy=0 1.571 0, axis 0 0 1, limit lower=-0.08 upper=0.02 effort=1000.0 velocity=0.5
- joint elbow_joint: axis (none) -> 1 0 0; limit (none) -> lower=-0.6 upper=0.6 effort=1000.0 velocity=0.5; origin xyz=0 0 0.4 rpy=1.571 0. 0. -> xyz=0 0 0.4 rpy=1.571 0 0
- joint wrist_joint: axis (none) -> 0 0 1
