Commit message: added sensor to urdf_advanced, added color check to advanced unit test

File: data/urdf/tests/merge_joint_box.urdf (robot description, URDF)
Before this commit: robot test_advanced, 7 links, 6 joints
Links:
- link finger_link_1: mass 10 -> None
- link finger_link_2: mass 10 -> None
- link link_1: geometry collision box size=0.1 0.1 0.8; visual box size=0.1 0.1 0.8
Joints:
- joint elbow_joint: type revolute -> fixed
- joint wrist_joint: type continuous -> fixed

File: data/urdf/tests/merge_joint_cylinder.urdf (robot description, URDF)
Before this commit: robot test_advanced, 7 links, 6 joints
Links:
- link finger_link_1: mass 10 -> None
- link finger_link_2: mass 10 -> None
Joints:
- joint elbow_joint: type revolute -> fixed
- joint wrist_joint: type continuous -> fixed
