Commit message: cleaned up unit test and test _urdfs. Material import broken though

File: data/urdf/tests/crash_test.urdf (robot description, URDF)
Before this commit: robot test_merge_joints, 7 links, 6 joints
Links:
- link finger_link_1: mass None -> 3
- link finger_link_2: mass None -> 3
- link link_1: geometry visual cylinder length=0.8 radius=.1
- link link_2: mass 10 -> None
- link palm_link: mass 10 -> None; geometry collision box size=0.2 .06 .06
Joints:
- joint elbow_joint: type fixed -> revolute
- joint finger_1_joint: limit lower=-0.02 upper=0.08 effort=1000.0 velocity=0.5 -> (none)
- joint wrist_joint: type fixed -> continuous

File: data/urdf/tests/test_basic.urdf (robot description, URDF)
Before this commit: robot test_basic, 7 links, 6 joints
Links:
- link base_link: geometry collision sphere radius=0.3; visual sphere radius=0.3
- link link_2: geometry collision capsule length=0.6 radius=.06; visual capsule length=0.6 radius=.06
