Commit message: modified some urdf test files

File: data/urdf/tests/test_basic.urdf (robot description, URDF)
Before this commit: robot test_basic, 7 links, 6 joints
Links:
- link finger_link_1: mass None -> 3
- link finger_link_2: mass None -> 3

File: data/urdf/tests/test_failure.urdf (robot description, URDF)
Before this commit: robot simple_gripper, 7 links, 6 joints
Links:
- link base_link: geometry collision box size=0.3 .3 .2; visual box size=0.3 .3 .2
- link finger_link_1: mass 10 -> 3
- link finger_link_2: mass 10 -> 3
- link link_1: geometry visual cylinder length=0.8 radius=.1
- link link_2: mass 10 -> None; geometry collision cylinder length=0.6 radius=.06; visual cylinder length=0.6 radius=.06
- link palm_link: mass 10 -> None
Joints:
- joint finger_1_joint: limit lower=-0.02 upper=0.08 effort=1000.0 velocity=0.5 -> (none)

Commit message: fixed cylinder visual/collision mesh rotation issue.

File: data/urdf/tests/test_basic.urdf (robot description, URDF)
Before this commit: robot test_basic, 7 links, 6 joints
Links:
- link base_link: geometry collision sphere radius=0.2; visual sphere radius=0.2

Commit message: Fix urdf import errors on TC, update to use ur10 mesh materials

File: data/urdf/tests/test_basic.urdf (robot description, URDF)
Before this commit: robot test_basic, 7 links, 6 joints
Links:
- link link_2: geometry collision cylinder length=0.6 radius=.06; visual cylinder length=0.6 radius=.06
