Commit message: Fix crash in urdf import, update urdf samples, update kaya urdf xacro

File: data/urdf/robots/kaya/urdf/kaya.urdf (robot description, URDF)
Before this commit: robot kaya, 49 links, 48 joints
Links:
- link assembly_battery: mass 4.266108 -> 0.4266108

File: data/urdf/robots/kaya/urdf/kaya.xacro (robot description, xacro)
@@ -69,5 +69,5 @@
     </visual>
 	<xacro:collision_box xyz="0.00033 -0.0127 0.00241" size="0.770 1.140 0.486"/>
-	<xacro:inertial_box xyz="0.00033 -0.0127 0.00241" size="0.770 1.140 0.486" rho="10"/>
+	<xacro:inertial_box xyz="0.00033 -0.0127 0.00241" size="0.770 1.140 0.486" rho="1"/>
   </link>
   <joint name="assembly_battery_joint" type="fixed">
