Commit message: update ur10 asset to be based off urdf-generated

File: data/urdf/robots/ur10/urdf/ur10_base.urdf (robot description, URDF)
Before this commit: robot UR10_CB3, 7 links, 6 joints
Links:
- removed link elbow_link
- added link forearm_link, mass 4.27; collision cylinder length=0.118 radius=0.047; collision cylinder length=0.126 radius=0.06
- link base_link: mass 20.0 -> 200.0; geometry collision cylinder length=0.03 radius=0.075; visual mesh filename=../meshes/ur10_base.obj scale=1.0
- link shoulder_link: geometry collision cylinder length=0.085 radius=0.075; collision cylinder length=0.17 radius=0.075
- link upper_arm_link: mass 4.27 -> 12.7; geometry collision cylinder length=0.136 radius=0.06; collision cylinder length=0.175 radius=0.075
- link wrist_1_link: geometry collision cylinder length=0.055 radius=0.047; collision cylinder length=0.118 radius=0.047
- link wrist_2_link: geometry collision cylinder length=0.054 radius=0.047; collision cylinder length=0.118 radius=0.047
- link wrist_3_link: geometry collision cylinder length=0.03 radius=0.047; visual mesh filename=../meshes/ur10_wrist_3.obj scale=1.0
Joints:
- removed joint elbow_joint
- removed joint wrist_3_joint
- added joint forearm_joint: type revolute, parent forearm_link, child wrist_1_link, origin xyz=0.572 0.116 0 rpy=0 0 0, axis 0 1 0, limit lower=-6.28318 upper=6.28318 effort=56.0 velocity=3.14159
- added joint upper_arm_joint: type revolute, parent upper_arm_link, child forearm_link, origin xyz=0.612 -0.128 0 rpy=0 0 0, axis 0 1 0, limit lower=-6.28318 upper=6.28318 effort=150.0 velocity=3.14159
- joint shoulder_lift_joint: child elbow_link -> upper_arm_link
- joint wrist_1_joint: axis 0 1 0 -> 0 0 -1; child wrist_1_link -> wrist_2_link; origin xyz=0.572 0.116 0 rpy=0 0 0 -> xyz=0 0 -0.116 rpy=0 0 0; parent upper_arm_link -> wrist_1_link
- joint wrist_2_joint: axis 0 0 -1 -> 0 1 0; child wrist_2_link -> wrist_3_link; origin xyz=0 0 -0.116 rpy=0 0 0 -> xyz=0 0.092 0 rpy=0 0 0; parent wrist_1_link -> wrist_2_link

Commit message: revert joint names on ur10 urdf

File: data/urdf/robots/ur10/urdf/ur10_base.urdf (robot description, URDF)
Before this commit: robot UR10_CB3, 7 links, 6 joints
Joints:
- removed joint forearm_joint
- removed joint upper_arm_joint
- added joint elbow_joint: type revolute, parent upper_arm_link, child forearm_link, origin xyz=0.612 -0.128 0 rpy=0 0 0, axis 0 1 0, limit lower=-6.28318 upper=6.28318 effort=150.0 velocity=3.14159
- added joint wrist_3_joint: type revolute, parent wrist_2_link, child wrist_3_link, origin xyz=0 0.092 0 rpy=0 0 0, axis 0 1 0, limit lower=-6.28318 upper=6.28318 effort=56.0 velocity=3.14159
- joint wrist_1_joint: axis 0 0 -1 -> 0 1 0; child wrist_2_link -> wrist_1_link; origin xyz=0 0 -0.116 rpy=0 0 0 -> xyz=0.572 0.116 0 rpy=0 0 0; parent wrist_1_link -> forearm_link
- joint wrist_2_joint: axis 0 1 0 -> 0 0 -1; child wrist_3_link -> wrist_2_link; origin xyz=0 0.092 0 rpy=0 0 0 -> xyz=0 0 -0.116 rpy=0 0 0; parent wrist_2_link -> wrist_1_link

Commit message: fix ur10 urdf import

File: data/urdf/robots/ur10/urdf/ur10_base.urdf (robot description, URDF)
Before this commit: robot UR10_CB3, 7 links, 6 joints
Links:
- link base_link: geometry collision cylinder length=0.03 radius=0.075; visual mesh filename=../meshes/ur10_base.obj scale=1 1 1
- link forearm_link: geometry collision cylinder length=0.118 radius=0.047; collision cylinder length=0.126 radius=0.06
- link shoulder_link: geometry collision cylinder length=0.085 radius=0.075; collision cylinder length=0.17 radius=0.075
- link upper_arm_link: geometry collision cylinder length=0.136 radius=0.06; collision cylinder length=0.175 radius=0.075
- link wrist_1_link: geometry collision cylinder length=0.055 radius=0.047; collision cylinder length=0.118 radius=0.047
- link wrist_2_link: geometry collision cylinder length=0.054 radius=0.047; collision cylinder length=0.118 radius=0.047
- link wrist_3_link: geometry collision cylinder length=0.03 radius=0.047; visual mesh filename=../meshes/ur10_wrist_3.obj scale=1 1 1
