Commit message: Cleanup extensions, Update Kit

File: data/urdf/robots/carter/urdf/carter.urdf (robot description, URDF)
Before this commit: robot carter, 6 links, 5 joints
Links:
- added link imu, mass .1; collision box size=.1 .1 .1
- link com_offset: geometry collision box size=.25 .25 .1
- link left_wheel_link: geometry collision sphere radius=0.240; visual mesh filename=package://carter/meshes/side_wheel.obj
- link rear_wheel_link: geometry collision sphere radius=.076; visual mesh filename=package://carter/meshes/caster_wheel.obj
- link right_wheel_link: geometry collision sphere radius=0.240; visual mesh filename=package://carter/meshes/side_wheel.obj
Joints:
- removed joint com_link
- added joint com_joint: type fixed, parent chassis_link, child com_offset, origin xyz=-.3 0 0 rpy=0 0 0, axis 0 1 0
- added joint imu_joint: type fixed, parent chassis_link, child imu, origin xyz=0 0 0 rpy=0 0 0, axis 0 1 0
