Commit message: Update Franka URDF: Joint 7 limits

File: source/extensions/omni.isaac.motion_generation/motion_policy_configs/franka/lula_franka_gen.urdf (robot description, URDF)
Before this commit: robot franka, 35 links, 34 joints
Joints:
- joint panda_joint7: limit lower=-1.8973 upper=1.8973 effort=12 velocity=2.6100 -> lower=-2.8973 upper=2.8973 effort=12 velocity=2.6100
