Commit message: Update UR10 URDFs to match UR10 Nucleus Assets

File: source/extensions/omni.isaac.motion_generation/motion_policy_configs/ur10/ur10_robot.urdf (robot description, URDF)
Before this commit: robot ur10, 11 links, 10 joints
Joints:
- joint ee_fixed_joint: origin xyz=0.0 0.0922 0.0 rpy=0.0 0.0 1.5707963267948966 -> xyz=0.0 0.0922 0.0 rpy=1.5707963267948966 0.0 1.5707963267948966

File: source/extensions/omni.isaac.motion_generation/motion_policy_configs/ur10/ur10_robot_suction.urdf (robot description, URDF)
Before this commit: robot ur10, 12 links, 11 joints
Joints:
- joint ee_fixed_joint: origin xyz=0.0 0.0922 0.0 rpy=0.0 0.0 1.5707963267948966 -> xyz=0.0 0.0922 0.0 rpy=1.5707963267948966 0.0 1.5707963267948966
