Commit message: ISIM-1983 reorganize ur10 ISIM-3119 Fix cobotta claw  ISIM-3118 Update single manipulator

File: source/extensions/isaacsim.robot_motion.motion_generation/motion_policy_configs/universal_robots/ur10/ur10_robot.urdf (robot description, URDF)
Before this commit: robot ur10, 11 links, 10 joints
Links:
- removed link base
- removed link tool0
- link base_link: mass 4.0 -> None; geometry 
- link ee_link: geometry 
- link forearm_link: mass 3.87 -> None; geometry 
- link shoulder_link: mass 7.778 -> None; geometry 
- link upper_arm_link: mass 12.93 -> None; geometry 
- link wrist_1_link: mass 1.96 -> None; geometry 
- link wrist_2_link: mass 1.96 -> None; geometry 
- link wrist_3_link: mass 0.202 -> None; geometry 
Joints:
- removed joint base_link-base_fixed_joint
- removed joint ee_fixed_joint
- removed joint wrist_3_link-tool0_fixed_joint
- added joint ee_joint: type fixed, parent wrist_3_link, child ee_link, origin xyz=-0. -0. -0. rpy=3.1415926 -1.57079638 0.
- joint elbow_joint: axis 0 1 0 -> 0. 0. 1.; limit lower=-3.141592653589793 upper=3.141592653589793 effort=150.0 velocity=3.15 -> lower=-3.1415927 upper=3.1415927 effort=150. velocity=3.1415927; origin xyz=0.0 -0.1719 0.612 rpy=0.0 0.0 0.0 -> xyz=-0.612 0. 0.  rpy=0. 0. 0.
- joint shoulder_lift_joint: axis 0 1 0 -> 0. 0. 1.; limit lower=-6.283185307179586 upper=6.283185307179586 effort=330.0 velocity=2.16 -> lower=-6.2831853 upper=6.2831853 effort=330. velocity=2.0943951; origin xyz=0.0 0.220941 0.0 rpy=0.0 1.5707963267948966 0.0 -> xyz=0. 0. 0. rpy=1.5707964 0. 0. 
- joint shoulder_pan_joint: axis 0 0 1 -> 0. 0. 1.; limit lower=-6.283185307179586 upper=6.283185307179586 effort=330.0 velocity=2.16 -> lower=-6.2831853 upper=6.2831853 effort=330. velocity=2.0943951; origin xyz=0.0 0.0 0.1273 rpy=0.0 0.0 0.0 -> xyz=0. 0. 0.1273 rpy=0. 0. -3.1415925
- joint wrist_1_joint: axis 0 1 0 -> 0. 0. 1.; limit lower=-6.283185307179586 upper=6.283185307179586 effort=54.0 velocity=3.2 -> lower=-6.2831853 upper=6.2831853 effort=56. velocity=3.1415927; origin xyz=0.0 0.0 0.5723 rpy=0.0 1.5707963267948966 0.0 -> xyz=-0.5723 0. 0.163941 rpy=0. 0. 0.
- joint wrist_2_joint: axis 0 0 1 -> 0. 0. 1.; limit lower=-6.283185307179586 upper=6.283185307179586 effort=54.0 velocity=3.2 -> lower=-6.2831853 upper=6.2831853 effort=56. velocity=3.1415927; origin xyz=0.0 0.1149 0.0 rpy=0.0 0.0 0.0 -> xyz=0. -0.1157 0.  rpy=1.5707964 0. 0. 
- joint wrist_3_joint: axis 0 1 0 -> 0. 0. 1.; limit lower=-6.283185307179586 upper=6.283185307179586 effort=54.0 velocity=3.2 -> lower=-6.2831853 upper=6.2831853 effort=56. velocity=3.1415927; origin xyz=0.0 0.0 0.1157 rpy=0.0 0.0 0.0 -> xyz=0. 0.0922 -0.  rpy=-1.5707964 -0.0000001 0.0000001
