Commit message: Fixes Fanuc CRX Asset Path + Joint names in the URDF files

File: source/extensions/isaacsim.robot_motion.motion_generation/motion_policy_configs/Fanuc/crx10ial/crx10ial.urdf (robot description, URDF)
Before this commit: robot fanuc_crx10ial, 10 links, 9 joints
Joints:
- removed joint joint_1
- removed joint joint_2
- removed joint joint_3
- removed joint joint_4
- removed joint joint_5
- removed joint joint_6
- removed joint joint_6-flange
- added joint J1: type revolute, parent base_link, child link_1, origin xyz=0 0 0.245 rpy=0 0 0, axis 0 0 1, limit lower=-3.141592653589793 upper=3.141592653589793 effort=0 velocity=2.0943951023931953
- added joint J2: type revolute, parent link_1, child link_2, origin xyz=0 0 0 rpy=0 0 0, axis 0 1 0, limit lower=-3.141592653589793 upper=3.141592653589793 effort=0 velocity=2.0943951023931953
- added joint J3: type revolute, parent link_2, child link_3, origin xyz=0 0 0.710 rpy=0 0 0, axis 0 -1 0, limit lower=-4.71238898038469 upper=4.71238898038469 effort=0 velocity=3.141592653589793
- added joint J4: type revolute, parent link_3, child link_4, origin xyz=0 0 0 rpy=0 0 0, axis -1 0 0, limit lower=-3.3161255787892263 upper=3.3161255787892263 effort=0 velocity=3.141592653589793
- added joint J5: type revolute, parent link_4, child link_5, origin xyz=0.540 -0.150 0 rpy=0 0 0, axis 0 -1 0, limit lower=-3.141592653589793 upper=3.141592653589793 effort=0 velocity=3.141592653589793
- added joint J6: type revolute, parent link_5, child link_6, origin xyz=0.160 0 0 rpy=0 0 0, axis -1 0 0, limit lower=-3.3161255787892263 upper=3.3161255787892263 effort=0 velocity=3.141592653589793
- added joint J6-flange: type fixed, parent link_6, child flange, origin xyz=0 0 0 rpy=0 0 0
